File: Kicad/Main_board.sch (KiCad schematic (older format))
At the start: 109 parts

Commit message: supprimé :        Kicad/CPU_board-cache.lib 	modifié :         Kicad/CPU_board.pro 	modifié :         Kicad/CPU_board.sch 	supprimé :        Kicad/CPU_board.sch-bak 	supprimé :        Kicad/Main_board-cache.lib 	modifié :         Kicad/Main_board.sch 	supprimé :        Kicad/Screen_board-cache.lib 	supprimé :        Kicad/Screen_board-rescue.dcm 	supprimé :        Kicad/Screen_board-rescue.lib 	supprimé :        Kicad/Screen_board.pro 	supprimé :        Kicad/Screen_board.sch 	supprimé :        Kicad/Screen_board.sch-bak
Parts:
- removed D? (x20): DIODE, symbol pspice:DIODE
- removed J?: Conn_01x17, symbol Connector_Generic:Conn_01x17
- added D33, D34, D35, D36, D37, D38, D39, D40, D41, D42, D43, D44, D45, D46, D47, D48, D49, D50, D51, D52: 1N4148, Diode_THT:D_DO-35_SOD27_P7.62mm_Horizontal, symbol Diode:1N4148
- added J1: Data, symbol Connector_Generic:Conn_02x08_Counter_Clockwise
- added J2: Power, symbol Connector_Generic:Conn_01x02
- gave numbers to parts that had none: 88
Connections:
- wire segments 276 -> 317
Other:
- note added: "Buttons matrix"
- note added: "Data & Power connectors"
- note added: "Step LED & Shift-register"
- note added: "Tempo LED & Shift-registers"
- moved on the sheet: D1, D10, D11, D12, D13, D14, D15, D16, D17, D18, D19, D2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
