File: Kicad/Main_board.kicad_pcb (KiCad board)
At the start: 2 copper layers, 213 x 128.5 mm, 110 parts, among them J1 Data, J2 Power, SW1 SW_Push, SW10 SW_Push, SW11 SW_Push, SW12 SW_Push, SW13 SW_Push, SW14 SW_Push, SW15 SW_Push, SW16 SW_Push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

Commit message: modifié :         Kicad/Main_board-cache.lib 	modifié :         Kicad/Main_board.kicad_pcb 	modifié :         Kicad/Main_board.net 	modifié :         Kicad/Main_board.sch 	nouveau fichier : Kicad/My_library/00_Mes_empreintes.pretty/7-Segment_2831AS.kicad_mod 	modifié :         Kicad/My_library/00_Mes_empreintes.pretty/DIP-16_Socket.kicad_mod 	nouveau fichier : Kicad/My_library/00_Mes_empreintes.pretty/IDC-Header_2x04.kicad_mod 	nouveau fichier : Kicad/My_library/00_Mes_empreintes.pretty/IDC-Header_2x05.kicad_mod 	modifié :         Kicad/My_library/00_Mes_empreintes.pretty/IDC-Header_2x08.kicad_mod 	modifié :         Kicad/My_library/00_Mes_empreintes.pretty/LED_5.0mm.kicad_mod 	nouveau fichier : Kicad/My_library/00_Mes_empreintes.pretty/RotaryEncoder.kicad_mod 	modifié :         Kicad/My_library/00_Mes_empreintes.pretty/SW_PUSH-12mm(deported).kicad_mod 	modifié :         Kicad/My_library/00_Mes_symboles.bck 	modifié :         Kicad/My_library/00_Mes_symboles.dcm 	modifié :         Kicad/My_library/00_Mes_symboles.lib 	nouveau fichier : Kicad/My_library/Encoders.lib 	nouveau fichier : "Kicad/My_library/Mes_mod\303\250les_3D/216-resistors-in-tht-series-e24-from-1ohm-to-910mohm-1.snapshot.3/Yageo CFR-25 Resistor Axial P7.62mm 1,0 MOhm.stp" 	nouveau fichier : "Kicad/My_library/Mes_mod\303\250les_3D/216-resistors-in-tht-series-e24-from-1ohm-to-910mohm-1.snapshot.3/Yageo CFR-25 Resistor Axial P7.62mm 1,0 Ohm.stp" 	nouveau fichier : "Kicad/My_library/Mes_mod\303\250les_3D/216-resistors-in-tht-series-e24-from-1ohm-to-910mohm-1.snapshot.3/Yageo CFR-25 Resistor Axial P7.62mm 1,0 kOhm.stp" 	nouveau fichier : "Kicad/My_library/Mes_mod\303\250les_3D/216-resistors-in-tht-series-e24-from-1ohm-to-910mohm-1.snapshot.3/Yageo CFR-25 Resistor Axial P7.62mm 1,1 MOhm.stp" 	nouveau fichier : "Kicad/My_library/Mes_mod\303\250les_3D/216-resistors-in-tht-series-e24-from-1ohm-to-910mohm-1.snapshot.3/Yageo CFR-25 Resistor Axial P7.62mm 1,1 Ohm.stp" 	nouveau fichier : "Kicad/My_library/Mes_mod\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
Parts:
- removed the J2 at (201.5, 50.5)
- added D53: LED, 00_Mes_empreintes:LED_5.0mm, F.Cu at (95.0, 66.0)
- added D54: LED, 00_Mes_empreintes:LED_5.0mm, F.Cu at (127.0, 66.0)
- added D55: LED, 00_Mes_empreintes:LED_5.0mm, F.Cu at (160.0, 66.0)
- added J1: Data & Power, 00_Mes_empreintes:IDC-Header_2x05, F.Cu at (152.5, 56.0)
- added J3: Data 3, 00_Mes_empreintes:IDC-Header_2x08, F.Cu at (177.5, 56.0)
- added R33: ?, 00_Mes_empreintes:Resistance, F.Cu at (172.0, 85.0)
- added R34: ?, 00_Mes_empreintes:Resistance, F.Cu at (177.0, 85.0)
- added R35: ?, 00_Mes_empreintes:Resistance, F.Cu at (167.0, 85.0)
- added R36: 50k, 00_Mes_empreintes:Resistance, F.Cu at (85.0, 79.0)
- added R37: 50k, 00_Mes_empreintes:Resistance, F.Cu at (117.0, 79.0)
- added R38: 50k, 00_Mes_empreintes:Resistance, F.Cu at (149.0, 79.0)
- added R39: 50k, 00_Mes_empreintes:Resistance, F.Cu at (85.0, 84.0)
- added R40: 50k, 00_Mes_empreintes:Resistance, F.Cu at (117.0, 84.0)
- added R41: 50k, 00_Mes_empreintes:Resistance, F.Cu at (149.0, 84.0)
- added R42: 220, 00_Mes_empreintes:Resistance, F.Cu at (95.0, 75.0)
- added R43: 220, 00_Mes_empreintes:Resistance, F.Cu at (127.0, 75.0)
- added R44: 220, 00_Mes_empreintes:Resistance, F.Cu at (159.0, 75.0)
- added SW21: Rotary_Encoder_Switch, 00_Mes_empreintes:RotaryEncoder, F.Cu at (75.0, 66.0)
- added SW22: Rotary_Encoder_Switch, 00_Mes_empreintes:RotaryEncoder, F.Cu at (107.0, 66.0)
- added SW23: Rotary_Encoder_Switch, 00_Mes_empreintes:RotaryEncoder, F.Cu at (139.0, 66.0)
- added SW24: Rotary_switch_8S.1P_(voltage_divider), 00_Mes_empreintes:SolderWirePad_1x03_Drill1.5mm, F.Cu at (109.0, 54.0)
- added U5: 7_segment_3_digit_2831AS, 00_Mes_empreintes:7-Segment_2831AS, F.Cu at (194.0, 71.0)
- J2: renamed from J1; value Data -> Data 2
- moved U4 26.0 mm to (60.5, 58.5)
- moved U3 25.5 mm to (53.0, 77.0), turned to 270 degrees
- moved J2 18.6 mm to (210.0, 56.0)
- moved U1 14.9 mm to (53.0, 50.0), turned to 270 degrees
- moved U2 4.95 mm to (53.0, 63.0), turned to 270 degrees
Connections:
- J2 pad 1: GND -> Selector_pin

Commit message: modifié :         Kicad/Main_board.kicad_pcb 	modifié :         README.md
Parts:
- moved U4 28.2 mm to (35.0, 70.5), turned to 90 degrees
- moved U2 27.7 mm to (35.0, 84.0), turned to 90 degrees
- moved U1 19.3 mm to (35.0, 57.0), turned to 90 degrees
- moved U3 18.4 mm to (68.5, 67.0), turned to 180 degrees
- moved J2 18.2 mm to (228.0, 53.5), turned to 90 degrees
- moved R42 10.0 mm to (95.0, 85.0), turned to 90 degrees
- moved R43 10.0 mm to (127.0, 85.0), turned to 90 degrees
- moved R44 10.0 mm to (159.0, 85.0), turned to 90 degrees
- moved D42 0.50 mm to (214.5, 99.5)
- moved D52 0.50 mm to (214.0, 145.5)
Routing:
- net Net-(R32-Pad2): track 0.00 -> 200.2 mm
- net Net-(R31-Pad2): track 0.00 -> 186.7 mm
- net Net-(R16-Pad2): track 0.00 -> 184.3 mm
- net Net-(R30-Pad2): track 0.00 -> 167.4 mm
- net Net-(R15-Pad2): track 0.00 -> 164.3 mm
- net Net-(R8-Pad2): track 0.00 -> 162.9 mm
- net Net-(R7-Pad2): track 0.00 -> 148.1 mm
- net Net-(R29-Pad2): track 0.00 -> 147.6 mm
- net Net-(R14-Pad2): track 0.00 -> 143.7 mm
- net Net-(R24-Pad2): track 0.00 -> 140.9 mm
- net Net-(R6-Pad2): track 0.00 -> 128.6 mm
- net Net-(R28-Pad2): track 0.00 -> 126.8 mm
- net Net-(R13-Pad2): track 0.00 -> 125.6 mm
- net Net-(R23-Pad2): track 0.00 -> 117.6 mm
- net Net-(R5-Pad2): track 0.00 -> 109.2 mm
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
Commit message: modifié :         Kicad/Main_board.kicad_pcb
Parts:
- moved J1 32.5 mm to (185.0, 56.0)
- moved J3 26.7 mm to (150.8, 56.0)
- moved R35 18.1 mm to (169.0, 67.0), turned to 0 degrees
- moved J2 17.2 mm to (211.0, 56.0), turned to 270 degrees
- moved R34 15.3 mm to (169.0, 72.0), turned to 0 degrees
- moved R33 8.54 mm to (169.0, 77.0), turned to 0 degrees
Routing:
- net GND: track 0.00 -> 847.4 mm, vias 0 -> 1
- net D: track 0.00 -> 427.3 mm
- net A: track 0.00 -> 354.8 mm, vias 0 -> 1
- net B: track 0.00 -> 326.3 mm, vias 0 -> 3
- net 3: track 0.00 -> 313.1 mm
- net C: track 0.00 -> 311.9 mm, vias 0 -> 1
- net +5V: track 5.00 -> 299.6 mm
- net 1: track 0.00 -> 253.0 mm
- net 4: track 0.00 -> 191.4 mm
- net 2: track 0.00 -> 174.1 mm
- net E: track 0.00 -> 148.6 mm
- net Net-(R25-Pad2): track 0.00 -> 74.1 mm
- net Latch_2: track 0.00 -> 66.6 mm
- net Clock_2: track 0.00 -> 66.0 mm
- net Net-(R17-Pad2): track 0.00 -> 52.0 mm
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